File: Amstrad_CPC_Keyboard/CPC6128/Amstrad_CPC6128_Keyboard.kicad_pcb (KiCad board)
At the start: 2 copper layers, 91 parts, among them J1 CP101_ODD, J2 CP101_EVEN, J3 CP102_A, J4 CP102_B, SW1 DEL, SW10 FOUR, SW11 THREE, SW12 E, SW13 W, SW14 S, SW15 D, SW16 C, SW17 X, SW18 SIX, SW19 FIVE, SW2 ONE, SW20 R, SW21 T, SW22 G, SW23 F, SW24 B, SW25 V, SW26 EIGHT, SW27 ZERO, SW28 CARAT, SW29 SEVEN, SW3 TWO, SW30 NINE, SW31 MINUS, SW32 U, SW33 O, SW34 @, SW35 Y, SW36 I, SW37 P, SW38 H, SW39 L, SW4 ESC, SW40 SEMI_COLON, SW41 J, SW42 K, SW43 COLON, SW44 N, SW45 M, SW46 /FORWSLASH/, SW47 SPACE, SW48 COMMA, SW49 DOT, SW5 Q, SW50 CLR, SW51 LEFT, SW52 UP, SW53 [, SW54 COPY, SW55 RIGHT, SW56 ENTER, SW57 NP_SEVEN, SW58 DOWN, SW59 ], SW6 TAB, SW60 NP_EIGHT, SW61 NP_NINE, SW62 NP_FOUR, SW63 NP_FIVE, SW64 NP_SIX, SW65 LH_SHIFT, SW66 NP_ONE, SW67 NP_THREE, SW68 \BACKSLASH\, SW69 NP_TWO, SW7 A, SW70 NP_ENTER, SW71 CTRL, SW72 NP_ZERO, SW73 NP_DOT, SW74 RH_SHIFT, SW8 CAPS_LOCK, SW9 Z

Commit message: CPC6128 keyboard updates
Parts:
- removed H7, H8: MountingHole, MountingHole:MountingHole_3.2mm_M3
- removed J2: CP101_EVEN, Connector_PinHeader_2.54mm:PinHeader_1x09_P2.54mm_Vertical
- removed J3: CP102_A, Connector_PinHeader_2.54mm:PinHeader_1x10_P2.54mm_Vertical
- removed J4: CP102_B, Connector_PinHeader_2.54mm:PinHeader_1x09_P2.54mm_Vertical
- added D1: LED, LED_THT:LED_D5.0mm, F.Cu at (329.2, 101.8)
- added KB70: NP_ENTER, PCM_Mounting_Keyboard_Stabilizer:Stabilizer_Cherry_MX_3.00u, F.Cu at (286.0, 198.3)
- added R1: R, Resistor_THT:R_Axial_DIN0207_L6.3mm_D2.5mm_P10.16mm_Horizontal, F.Cu at (344.4, 109.4)
- added SW75: SW_SPST, Button_Switch_THT:SW_Slide_SPDT_Straight_CK_OS102011MS2Q, F.Cu at (346.4, 101.8)
- J1: value CP101_ODD -> POWER; footprint Connector_PinHeader_2.54mm:PinHeader_1x10_P2.54mm_Vertical -> Connector_PinHeader_2.54mm:PinHeader_1x02_P2.54mm_Vertical; moved to F.Cu
- SW1: footprint PCM_Switch_Keyboard_Cherry_MX:SW_Cherry_MX_PCB_1.25u -> PCM_Switch_Keyboard_Cherry_MX:SW_Cherry_MX_PCB_1.00u
- SW54, SW71: footprint PCM_Switch_Keyboard_Cherry_MX:SW_Cherry_MX_PCB_1.00u -> PCM_Switch_Keyboard_Cherry_MX:SW_Cherry_MX_PCB_2.50u
- SW6: footprint PCM_Switch_Keyboard_Cherry_MX:SW_Cherry_MX_PCB_1.75u -> PCM_Switch_Keyboard_Cherry_MX:SW_Cherry_MX_PCB_1.50u
- SW65: footprint PCM_Switch_Keyboard_Cherry_MX:SW_Cherry_MX_PCB_2.25u -> PCM_Switch_Keyboard_Cherry_MX:SW_Cherry_MX_PCB_2.00u
- SW70: footprint PCM_Switch_Keyboard_Cherry_MX:SW_Cherry_MX_PCB_1.00u -> PCM_Switch_Keyboard_Cherry_MX:SW_Cherry_MX_PCB_3.00u
- SW8: footprint PCM_Switch_Keyboard_Cherry_MX:SW_Cherry_MX_PCB_2.00u -> PCM_Switch_Keyboard_Cherry_MX:SW_Cherry_MX_PCB_1.75u
- moved J1 322.9 mm to (359.7, 106.9), turned to 180 degrees
- moved SW51 120.6 mm to (324.1, 198.3)
- moved SW55 120.6 mm to (362.2, 198.3)
- moved SW52 120.6 mm to (343.2, 179.3)
- moved SW58 101.8 mm to (343.2, 198.3)
- moved SW70 97.2 mm to (286.0, 198.3)
- moved H3 68.8 mm to (209.8, 106.9)
- moved H5 59.5 mm to (369.8, 106.9)
- moved H1 56.2 mm to (32.0, 106.9)
- moved H4 42.9 mm to (207.3, 213.6)
- moved H6 21.2 mm to (369.8, 213.6)
- moved SW57 19.2 mm to (324.1, 122.1)
- moved SW60 19.2 mm to (343.2, 122.1)
- moved SW62 19.2 mm to (324.1, 141.2)
- moved SW63 19.2 mm to (343.2, 141.2)
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Connections:
- J1 pad 1: KB_1 -> /+5V
- J1 pad 2: KB_3 -> /GND
Other:
- board text removed: "1"
- board text removed: "19"
