File: Amstrad_CPC_Keyboard/CPC6128/Amstrad_CPC6128_Keyboard.kicad_sch (KiCad schematic)
At the start: 91 parts, among them J1 CP101_ODD, J2 CP101_EVEN, J3 CP102_A, J4 CP102_B, SW1 DEL, SW10 FOUR, SW11 THREE, SW12 E, SW13 W, SW14 S, SW15 D, SW16 C, SW17 X, SW18 SIX, SW19 FIVE, SW2 ONE, SW20 R, SW21 T, SW22 G, SW23 F, SW24 B, SW25 V, SW26 EIGHT, SW27 ZERO, SW28 CARAT, SW29 SEVEN, SW3 TWO, SW30 NINE, SW31 MINUS, SW32 U, SW33 O, SW34 @, SW35 Y, SW36 I, SW37 P, SW38 H, SW39 L, SW4 ESC, SW40 SEMI_COLON, SW41 J, SW42 K, SW43 COLON, SW44 N, SW45 M, SW46 /FORWSLASH/, SW47 SPACE, SW48 COMMA, SW49 DOT, SW5 Q, SW50 CLR, SW51 LEFT, SW52 UP, SW53 [, SW54 COPY, SW55 RIGHT, SW56 ENTER, SW57 NP_SEVEN, SW58 DOWN, SW59 ], SW6 TAB, SW60 NP_EIGHT, SW61 NP_NINE, SW62 NP_FOUR, SW63 NP_FIVE, SW64 NP_SIX, SW65 LH_SHIFT, SW66 NP_ONE, SW67 NP_THREE, SW68 \BACKSLASH\, SW69 NP_TWO, SW7 A, SW70 NP_ENTER, SW71 CTRL, SW72 NP_ZERO, SW73 NP_DOT, SW74 RH_SHIFT, SW8 CAPS_LOCK, SW9 Z

Commit message: CPC6128 keyboard updates
Parts:
- removed H7, H8: MountingHole, MountingHole:MountingHole_3.2mm_M3, symbol Mechanical:MountingHole
- removed J1: CP101_ODD, Connector_PinHeader_2.54mm:PinHeader_1x10_P2.54mm_Vertical, symbol Connector_Generic:Conn_01x10
- removed J2: CP101_EVEN, Connector_PinHeader_2.54mm:PinHeader_1x09_P2.54mm_Vertical, symbol Connector_Generic:Conn_01x09
- removed J3: CP102_A, Connector_PinHeader_2.54mm:PinHeader_1x10_P2.54mm_Vertical, symbol Connector_Generic:Conn_01x10
- removed J4: CP102_B, Connector_PinHeader_2.54mm:PinHeader_1x09_P2.54mm_Vertical, symbol Connector_Generic:Conn_01x09
- added D1: LED, LED_THT:LED_D5.0mm, symbol Device:LED
- added J1: POWER, Connector_PinHeader_2.54mm:PinHeader_1x02_P2.54mm_Vertical, symbol Connector_Generic:Conn_01x02
- added KB70: NP_ENTER, PCM_Mounting_Keyboard_Stabilizer:Stabilizer_Cherry_MX_3.00u, symbol Clueless_Engineer:Stabiliser
- added R1: R, Resistor_THT:R_Axial_DIN0207_L6.3mm_D2.5mm_P10.16mm_Horizontal, symbol Device:R
- added SW75: SW_SPST, Button_Switch_THT:SW_Slide_SPDT_Straight_CK_OS102011MS2Q, symbol Switch:SW_SPST
- SW1: footprint PCM_Switch_Keyboard_Cherry_MX:SW_Cherry_MX_PCB_1.25u -> PCM_Switch_Keyboard_Cherry_MX:SW_Cherry_MX_PCB_1.00u
- SW54, SW71: footprint PCM_Switch_Keyboard_Cherry_MX:SW_Cherry_MX_PCB_1.00u -> PCM_Switch_Keyboard_Cherry_MX:SW_Cherry_MX_PCB_2.50u
- SW6: footprint PCM_Switch_Keyboard_Cherry_MX:SW_Cherry_MX_PCB_1.75u -> PCM_Switch_Keyboard_Cherry_MX:SW_Cherry_MX_PCB_1.50u
- SW65: footprint PCM_Switch_Keyboard_Cherry_MX:SW_Cherry_MX_PCB_2.25u -> PCM_Switch_Keyboard_Cherry_MX:SW_Cherry_MX_PCB_2.00u
- SW70: footprint PCM_Switch_Keyboard_Cherry_MX:SW_Cherry_MX_PCB_1.00u -> PCM_Switch_Keyboard_Cherry_MX:SW_Cherry_MX_PCB_3.00u
- SW8: footprint PCM_Switch_Keyboard_Cherry_MX:SW_Cherry_MX_PCB_2.00u -> PCM_Switch_Keyboard_Cherry_MX:SW_Cherry_MX_PCB_1.75u
Connections:
- new net: D1.1 (K), SW75.2 (B)
- new net: D1.2 (A), R1.1
- new net +5V: J1.1 (Pin_1), R1.2
- new net GND: J1.2 (Pin_2), SW75.1 (A)
Other:
- moved on the sheet: H5
