File: Amstrad_CPC_Keyboard/CPC6128/CherryMX/Amstrad_CPC6128_Keyboard.kicad_sch (KiCad schematic)
At the start: 90 parts, among them J1 POWER, SW1 DEL, SW10 FOUR, SW11 THREE, SW12 E, SW13 W, SW14 S, SW15 D, SW16 C, SW17 X, SW18 SIX, SW19 FIVE, SW2 ONE, SW20 R, SW21 T, SW22 G, SW23 F, SW24 B, SW25 V, SW26 EIGHT, SW27 ZERO, SW28 CARAT, SW29 SEVEN, SW3 TWO, SW30 NINE, SW31 MINUS, SW32 U, SW33 O, SW34 @, SW35 Y, SW36 I, SW37 P, SW38 H, SW39 L, SW4 ESC, SW40 SEMI_COLON, SW41 J, SW42 K, SW43 COLON, SW44 N, SW45 M, SW46 /FORWSLASH/, SW47 SPACE, SW48 COMMA, SW49 DOT, SW5 Q, SW50 CLR, SW51 LEFT, SW52 UP, SW53 [, SW54 COPY, SW55 RIGHT, SW56 ENTER, SW57 NP_SEVEN, SW58 DOWN, SW59 ], SW6 TAB, SW60 NP_EIGHT, SW61 NP_NINE, SW62 NP_FOUR, SW63 NP_FIVE, SW64 NP_SIX, SW65 LH_SHIFT, SW66 NP_ONE, SW67 NP_THREE, SW68 \BACKSLASH\, SW69 NP_TWO, SW7 A, SW70 NP_ENTER, SW71 CTRL, SW72 NP_ZERO, SW73 NP_DOT, SW74 RH_SHIFT, SW75 SW_SPST, SW8 CAPS_LOCK, SW9 Z

Commit message: Reorganise CPC projects
Parts:
- removed KB56: ENTER, PCM_Mounting_Keyboard_Stabilizer:Stabilizer_Cherry_MX_2.00u, symbol Clueless_Engineer:Stabiliser
- removed KB65: LH_SHIFT, PCM_Mounting_Keyboard_Stabilizer:Stabilizer_Cherry_MX_2.00u, symbol Clueless_Engineer:Stabiliser
- removed KB70: NP_ENTER, PCM_Mounting_Keyboard_Stabilizer:Stabilizer_Cherry_MX_3.00u, symbol Clueless_Engineer:Stabiliser
- removed KB74: RH_SHIFT, PCM_Mounting_Keyboard_Stabilizer:Stabilizer_Cherry_MX_2.00u, symbol Clueless_Engineer:Stabiliser
- removed KB8: CAPS_LOCK, PCM_Mounting_Keyboard_Stabilizer:Stabilizer_Cherry_MX_2.00u, symbol Clueless_Engineer:Stabiliser
- SW28: value CARAT -> ^CARAT^
- SW31: value MINUS -> -MINUS-
- SW34: value @ -> @AT@
- SW40: value SEMI_COLON -> ;SEMI_COLON;
- SW43: value COLON -> :COLON:
- SW48: value COMMA -> ,COMMA,
- SW49: value DOT -> .DOT.
