File: Amstrad_CPC_Keyboard/CPC6128/Tactile/Amstrad_CPC6128_Keyboard.kicad_pcb (KiCad board)
At the start: 2 copper layers, 293 x 99 mm, 84 parts, among them J2 Keyboard CP002, J3 CP001, SW1 DEL, SW10 FOUR, SW11 THREE, SW12 E, SW13 W, SW14 S, SW15 D, SW16 C, SW17 X, SW18 SIX, SW19 FIVE, SW2 ONE, SW20 R, SW21 T, SW22 G, SW23 F, SW24 B, SW25 V, SW26 EIGHT, SW27 ZERO, SW28 ^CARAT^, SW29 SEVEN, SW3 TWO, SW30 NINE, SW31 -MINUS-, SW32 U, SW33 O, SW34 @AT@, SW35 Y, SW36 I, SW37 P, SW38 H, SW39 L, SW4 ESC, SW40 ;SEMI_COLON;, SW41 J, SW42 K, SW43 :COLON:, SW44 N, SW45 M, SW46 /FORWSLASH/, SW47 SPACE, SW48 ,COMMA,, SW49 .DOT., SW5 Q, SW50 CLR, SW51 LEFT, SW52 UP, SW53 [, SW54 COPY, SW55 RIGHT, SW56 ENTER, SW57 NP_SEVEN, SW58 DOWN, SW59 ], SW6 TAB, SW60 NP_EIGHT, SW61 NP_NINE, SW62 NP_FOUR, SW63 NP_FIVE, SW64 NP_SIX, SW65 LH_SHIFT, SW66 NP_ONE, SW67 NP_THREE, SW68 \BACKSLASH\, SW69 NP_TWO, SW7 A, SW70 NP_ENTER, SW71 CTRL, SW72 NP_ZERO, SW73 NP_DOT, SW74 RH_SHIFT, SW75 SW_SPDT, SW8 CAPS_LOCK, SW9 Z

Commit message: Finalised Rev. A of tactile keyboard design
Parts:
- removed J2: Keyboard CP002, Connector_PinHeader_2.54mm:PinHeader_1x19_P2.54mm_Vertical
- added H4: MountingHole, MountingHole:MountingHole_3.2mm_M3, F.Cu at (62.8, 188.0)
- added H6: MountingHole, MountingHole:MountingHole_3.2mm_M3, F.Cu at (196.8, 188.0)
- added J1: CP002, Connector_PinHeader_2.54mm:PinHeader_1x10_P2.54mm_Vertical, F.Cu at (64.1, 99.0)
- added J4: CP003, Connector_PinHeader_2.54mm:PinHeader_1x09_P2.54mm_Vertical, F.Cu at (92.0, 99.0)
- SW1: value DEL -> DEL (79)
- SW10: value FOUR -> FOUR (56)
- SW11: value THREE -> THREE (57)
- SW12: value E -> E (58)
- SW13: value W -> W (59)
- SW14: value S -> S (60)
- SW15: value D -> D (61)
- SW16: value C -> C (62)
- SW17: value X -> X (63)
- SW18: value SIX -> SIX (48)
- SW19: value FIVE -> FIVE (49)
- SW2: value ONE -> ONE (64)
- SW20: value R -> R (50)
- SW21: value T -> T (51)
- SW22: value G -> G (52)
- SW23: value F -> F (53)
- SW24: value B -> B (54)
- SW25: value V -> V (55)
- SW26: value EIGHT -> EIGHT (40)
- SW27: value ZERO -> ZERO (32)
- SW28: value ^CARAT^ -> ^CARAT^ (24)
- SW29: value SEVEN -> SEVEN (41)
- SW3: value TWO -> TWO (65)
- SW30: value NINE -> NINE (33)
- SW31: value -MINUS- -> -MINUS- (25)
- SW32: value U -> U (42)
- SW33: value O -> O (34)
- SW34: value @AT@ -> @AT@ (26)
- SW35: value Y -> Y (43)
- SW36: value I -> I (35)
- SW37: value P -> P (27)
- SW38: value H -> H (44)
- SW39: value L -> L (36)
- SW4: value ESC -> ESC (66)
- SW40: value ;SEMI_COLON; -> ;SEMI_COLON; (28)
- SW41: value J -> J (45)
- SW42: value K -> K (37)
- SW43: value :COLON: -> :COLON: (29)
- SW44: value N -> N (46)
- SW45: value M -> M (38)
- SW46: value /FORWSLASH/ -> /FORWSLASH/ (30)
- SW47: value SPACE -> SPACE (47)
- SW48: value ,COMMA, -> ,COMMA, (39)
- SW49: value .DOT. -> .DOT. (31)
- SW5: value Q -> Q (67)
- SW50: value CLR -> CLR (16)
- SW51: value LEFT -> LEFT (08)
- SW52: value UP -> UP (00)
- SW53: value [ -> [ (17)
- SW54: value COPY -> COPY (09)
- SW55: value RIGHT -> RIGHT (01)
- SW56: value ENTER -> ENTER (18)
- SW57: value NP_SEVEN -> ƒ7 (10)
- SW58: value DOWN -> DOWN (02)
- SW59: value ] -> ] (19)
- SW6: value TAB -> TAB (68)
- SW60: value NP_EIGHT -> ƒ8 (11)
- SW61: value NP_NINE -> ƒ9 (03)
- SW62: value NP_FOUR -> ƒ4 (20)
- SW63: value NP_FIVE -> ƒ5 (12)
- SW64: value NP_SIX -> ƒ6 (04)
- SW65: value LH_SHIFT -> LH_SHIFT (21)
- SW66: value NP_ONE -> ƒ1 (13)
- SW67: value NP_THREE -> ƒ3 (05)
- SW68: value \BACKSLASH\ -> \BACKSLASH\ (22)
- SW69: value NP_TWO -> ƒ2 (14)
- SW7: value A -> A (69)
- SW70: value NP_ENTER -> ENTER (06)
- SW71: value CTRL -> CTRL (23)
- SW72: value NP_ZERO -> ƒ0 (15)
- SW73: value NP_DOT -> .DOT. (07)
- SW74: value RH_SHIFT -> RH_SHIFT (21)
- SW8: value CAPS_LOCK -> CAPS_LOCK (70)
- SW9: value Z -> Z (71)
- moved SW55 74.5 mm to (294.8, 180.0)
- moved SW52 71.8 mm to (278.8, 164.0)
- moved SW51 70.0 mm to (262.8, 180.0)
- moved SW56 65.1 mm to (278.8, 141.0)
- moved SW66 56.6 mm to (302.8, 148.0)
- moved J3 56.6 mm to (334.7, 107.0)
- moved LS1 56.6 mm to (293.6, 103.6)
- moved SW75 56.6 mm to (316.7, 104.4)
- moved H1 56.6 mm to (347.8, 108.0)
- moved H2 56.6 mm to (62.8, 108.0)
- moved H3 56.6 mm to (196.8, 99.0)
- moved H5 56.6 mm to (347.8, 188.0)
- moved R1 56.6 mm to (299.0, 107.6)
- moved SW1 56.6 mm to (286.8, 116.0)
- moved SW10 56.6 mm to (126.8, 116.0)
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Connections:
- net KB_10 renamed X8
- net KB_11 renamed Y9
- net KB_12 renamed Y8
- net KB_13 renamed Y7
- net KB_14 renamed Y6
- net KB_15 renamed Y5
- net KB_16 renamed Y4
- net KB_17 renamed Y3
- net KB_18 renamed Y2
- net KB_19 renamed Y1
- net KB_3 renamed X1
- net KB_4 renamed X2
- net KB_5 renamed X3
- net KB_6 renamed X4
- net KB_7 renamed X5
- net KB_8 renamed X6
- net KB_9 renamed X7
- SW1 pad 1: KB_1 -> X9
- SW1 pad 2: KB_2 -> Y10
Routing:
- net X9: track 0.00 -> 260.6 mm
- net KB_1: track 260.6 -> 0.00 mm
- net Y10: track 0.00 -> 260.3 mm
- net KB_2: track 260.3 -> 0.00 mm
- net Y7: track 282.5 -> 248.9 mm
- net Y5: track 336.6 -> 303.1 mm
- net X2: track 353.2 -> 381.5 mm
- net Y4: track 349.2 -> 322.1 mm
- net X1: track 316.7 -> 336.3 mm
- net X6: track 395.5 -> 378.5 mm
- net Y1: track 463.6 -> 450.6 mm
- net X7: track 434.0 -> 425.2 mm
- net X3: track 357.8 -> 362.4 mm
- net Y3: track 568.9 -> 572.8 mm
- net Y2: track 413.5 -> 410.6 mm
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Other:
- board text added: "(KEY NUMBERS IN BRACKETS)"
- board text added: "CP002"
- board text added: "CP003"
- board text added: "OFF/ON"
- board text added: "X3 X2 X1 Y10 X9"
- board text added: "X6 X5 X4"
- board text added: "X6 X7 X8"
- board text added: "X8 X7"
- board text added: "Y1 Y2"
- board text added: "Y3 Y4 Y5"
- board text added: "Y6 Y7 Y8 Y9"
- board text added: "Y9"
- board text removed: "OFF / ON"
- board text removed: "X6 X7"
- board text removed: "X8 X9"
