File: Amstrad_CPC_Keyboard/CPC6128/Tactile_12mm/Amstrad_Tactile-12mm_Keyboard.kicad_pcb (KiCad board)
At the start: 2 copper layers, 293 x 99 mm, 87 parts, among them J1 CP002, J3 CP001, J4 CP003, SW1 DEL (79), SW10 FOUR (56), SW11 THREE (57), SW12 E (58), SW13 W (59), SW14 S (60), SW15 D (61), SW16 C (62), SW17 X (63), SW18 SIX (48), SW19 FIVE (49), SW2 ONE (64), SW20 R (50), SW21 T (51), SW22 G (52), SW23 F (53), SW24 B (54), SW25 V (55), SW26 EIGHT (40), SW27 ZERO (32), SW28 ^CARAT^ (24), SW29 SEVEN (41), SW3 TWO (65), SW30 NINE (33), SW31 -MINUS- (25), SW32 U (42), SW33 O (34), SW34 @AT@ (26), SW35 Y (43), SW36 I (35), SW37 P (27), SW38 H (44), SW39 L (36), SW4 ESC (66), SW40 ;SEMI_COLON; (28), SW41 J (45), SW42 K (37), SW43 :COLON: (29), SW44 N (46), SW45 M (38), SW46 /FORWSLASH/ (30), SW47 SPACE (47), SW48 ,COMMA, (39), SW49 .DOT. (31), SW5 Q (67), SW50 CLR (16), SW51 LEFT (08), SW52 UP (00), SW53 [ (17), SW54 COPY (09), SW55 RIGHT (01), SW56 ENTER (18), SW57 ƒ7 (10), SW58 DOWN (02), SW59 ] (19), SW6 TAB (68), SW60 ƒ8 (11), SW61 ƒ9 (03), SW62 ƒ4 (20), SW63 ƒ5 (12), SW64 ƒ6 (04), SW65 LH_SHIFT (21), SW66 ƒ1 (13), SW67 ƒ3 (05), SW68 \BACKSLASH\ (22), SW69 ƒ2 (14), SW7 A (69), SW70 ENTER (06), SW71 CTRL (23), SW72 ƒ0 (15), SW73 .DOT. (07), SW74 RH_SHIFT (21), SW75 SW_SPDT, SW8 CAPS_LOCK (70), SW9 Z (71)

Commit message: Added 6mm tactile design
Parts:
- removed J4: CP003, Connector_PinHeader_2.54mm:PinHeader_1x09_P2.54mm_Vertical
- added J2: CP003, Connector_PinHeader_2.54mm:PinHeader_1x10_P2.54mm_Vertical, F.Cu at (90.1, 98.3)
- J1: footprint Connector_PinHeader_2.54mm:PinHeader_1x10_P2.54mm_Vertical -> Connector_PinHeader_2.54mm:PinHeader_1x09_P2.54mm_Vertical
- moved J1 0.92 mm to (64.7, 98.3)
Connections:
- J1 pad 1: X9 -> X1
- J1 pad 2: Y10 -> X2
- J1 pad 3: X1 -> X3
- J1 pad 4: X2 -> X4
- J1 pad 5: X3 -> X5
- J1 pad 6: X4 -> X6
- J1 pad 7: X5 -> X7
- J1 pad 8: X6 -> X8
- J1 pad 9: X7 -> X9
Routing:
- net X4: track 414.4 -> 349.9 mm
- net Y6: track 324.3 -> 289.4 mm
- net Y8: track 248.8 -> 216.7 mm
- net Y10: track 260.3 -> 233.8 mm
- net X9: track 260.6 -> 240.1 mm
- net X6: track 378.5 -> 387.0 mm
- net X7: track 425.2 -> 433.1 mm
- net X8: track 377.6 -> 385.4 mm
- net X5: track 397.5 -> 405.2 mm
- net Y5: track 303.1 -> 298.9 mm
- net Y9: track 257.0 -> 253.8 mm
- net X3: track 362.4 -> 364.2 mm, vias 0 -> 1
- net Y4: track 322.1 -> 320.8 mm
- net X1: track 336.3 -> 337.1 mm
Other:
- board text added: "X1 X2 X3 X4 X5 X6 X7 X8 X9"
- board text added: "Y10 Y9 Y8 Y7 Y6 Y5 Y4 Y3 Y2 Y1"
- board text removed: "X3 X2 X1 Y10 X9"
- board text removed: "X4 X5"
- board text removed: "X6 X5 X4"
- board text removed: "X6 X7 X8"
- board text removed: "X8 X7"
- board text removed: "X9 Y10 X1 X2 X3"
- board text removed: "Y1 Y2"
- board text removed: "Y2 Y1"
- board text removed: "Y3 Y4 Y5"
- board text removed: "Y4 Y3"
- board text removed: "Y6 Y5"
- board text removed: "Y6 Y7 Y8 Y9"
- board text removed: "Y8 Y7"
- board text removed: "Y9"
