File: VGA4CPC_Brett/RevC/VGA4CPC_Brett_RevC.kicad_pcb (KiCad board)
At the start: 2 copper layers, 95 x 70 mm, 49 parts, among them J1 CPC VIDEO IN, J2 LUM OUT, J3 +5V IN, J4 VFREQ, J5 SPARE GPIO, J6 VGA OUT, SW1 RESET, SW2 WACKED, U1 RASPBERRY PI PICO2, U2 74LVC245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

Commit message: Added +3.3V on spare GPIO header
Parts:
- J5: footprint Connector_PinHeader_2.54mm:PinHeader_1x06_P2.54mm_Vertical -> Connector_PinHeader_2.54mm:PinHeader_1x07_P2.54mm_Vertical
- moved J5 0.51 mm to (146.7, 123.2)
Routing:
- net /UPPER: track 45.8 -> 65.2 mm, vias 0 -> 2
- net /LOWER: track 44.8 -> 62.9 mm, vias 0 -> 2
- net GND: track 23.3 -> 35.6 mm, vias 1 -> 4
- net +3.3V: track 150.2 -> 153.0 mm
Other:
- board text added: "+3.3V"
