File: CPC_DIN-to-VGA/CPC_DIN-to-VGA.kicad_sch (KiCad schematic)
At the start: 5 parts, among them J1 DIN-6, J2 CPC PLUS VIDEO IN, J3 CPC PLUS AUDIO OUT, J4 VGA OUT, J5 LUM OUT

Commit message: Updated PCB text to "15KHz VGA OUT"
Parts:
- J4: value VGA OUT -> 15KHz VGA OUT
Changed lines of the file:
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@@
 			)
 		)
-		(property "Value" "VGA OUT"
+		(property "Value" "15KHz VGA OUT"
 			(at 172.72 20.32 0)
 			(effects
