File: VGA4CPC_Brett/Comparator_Board/Comparator_Board.kicad_sch (KiCad schematic)
At the start: 18 parts, among them J1 INPUT, J2 OUTPUT, U1 TLV3232, U2 TLV3232, U3 TLV3232

Commit message: Finalised voltage divider resistor values
Parts:
- R1: value 17KΩ -> 18KΩ
- R2: value 3KΩ -> 3.3KΩ
- R3: value 19KΩ -> 18KΩ
